Commit message: robot sensors

File: src/my_robot/urdf/my_robot.xacro (robot description, xacro)
@@ -1,16 +1,25 @@
 <?xml version='1.0'?>
 <robot name="my_robot" xmlns:xacro="http://www.ros.org/wiki/xacro">
+  <material name="blue">
+    <color rgba="0 0 0.8 1"/>
+  </material>
+  <material name="green">
+    <color rgba="0 1 0 1"/>
+  </material>
+  <material name="red">
+    <color rgba="1 0 0 1"/>
+  </material>
   <link name="robot_footprint"></link>
   <link name='chassis'>
-	<pose>0 0 0.1 0 0 0</pose>
-    <inertial>
-    	<mass value="15.0"/>
-    	<origin xyz="0.0 0 0" rpy=" 0 0 0"/>
-    	<inertia
+	  <pose>0 0 0.1 0 0 0</pose>
+      <inertial>
+    	  <mass value="15.0"/>
+    	  <origin xyz="0.0 0 0" rpy=" 0 0 0"/>
+    	  <inertia
           ixx="0.1" ixy="0" ixz="0"
           iyy="0.1" iyz="0"
           izz="0.1"
-      	/>
-    </inertial>
+      	  />
+      </inertial>
     <collision name='collision'>
       <origin xyz="0 0 0" rpy=" 0 0 0"/>
@@ -24,4 +33,5 @@
         <box size=".4 .2 .1"/>
       </geometry>
+      <material name="blue"/>
     </visual>
     <collision name='back_caster_collision'>
@@ -51,5 +61,5 @@
   </link>
   <link name="left_wheel">
-	<inertial>
+	  <inertial>
     	<mass value="5.0"/>
     	<origin xyz="0.0 0 0" rpy=" 0 1.5707 1.5707"/>
@@ -60,11 +70,12 @@
       	/>
     </inertial>
-	<visual name='left_wheel'>
+	  <visual name='left_wheel'>
       <origin xyz="0 0 0" rpy=" 0 1.5707 1.5707"/>
       <geometry>
         <cylinder radius="0.1" length="0.05"/>
       </geometry>
+      <material name="green"/>
     </visual>
-	<collision name='left_wheel'>
+	  <collision name='left_wheel'>
       <origin xyz="0 0 0" rpy=" 0 1.5707 1.5707"/>
       <geometry>
@@ -74,5 +85,5 @@
   </link>
   <link name="right_wheel">
-	<inertial>
+	  <inertial>
     	<mass value="5.0"/>
     	<origin xyz="0.0 0 0" rpy=" 0 1.5707 1.5707"/>
@@ -83,14 +94,55 @@
       	/>
     </inertial>
-	<visual name='right_wheel'>
+	  <visual name='right_wheel'>
       <origin xyz="0 0 0" rpy=" 0 1.5707 1.5707"/>
       <geometry>
         <cylinder radius="0.1" length="0.05"/>
       </geometry>
+      <material name="green"/>
     </visual>
-	<collision name='right_wheel'>
+	  <collision name='right_wheel'>
       <origin xyz="0 0 0" rpy=" 0 1.5707 1.5707"/>
       <geometry>
         <cylinder radius="0.1" length="0.05"/>
+      </geometry>
+    </collision>
+  </link>
+  <link name="camera">
+    <box_inertia x="0.05" y="0.05" z="0.05" m="0.1" />
+    <inertial>
+      <mass value="0.1"/>
+      <origin xyz="0.0 0.0 0.0" rpy="0.0 0.0 0.0"/>
+      <inertia ixx="1e-6" ixy="0" ixz="0" iyy="1e-6" iyz="0" izz="1e-6"/>
+    </inertial>
+    <visual name="camera">
+      <origin xyz="0.0 0.0 0.0" rpy="0.0 0.0 0.0"/>
+      <geometry>
+        <box size="0.05 0.05 0.05"/>
+      </geometry>
+      <material name="red"/>
+    </visual>
+    <collision>
+      <origin xyz="0.0 0.0 0.0" rpy="0.0 0.0 0.0"/>
+      <geometry>
+        <box size="0.05 0.05 0.05"/>
+      </geometry>
+    </collision>
+  </link>
+  <link name="hokuyo">
+    <inertial>
+      <origin xyz="0.0 0.0 0.0" rpy="0.0 0.0 0.0"/>
+      <mass value="1e-5"/>
+      <inertia ixx="1e-6" ixy="0" ixz="0" iyy="1e-6" iyz="0" izz="1e-6"/>
+    </inertial>
+    <visual name="hokuyo">
+      <origin xyz="0.0 0.0 0.0" rpy="0.0 0.0 0.0"/>
+      <geometry>
+        <mesh filename="package://my_robot/meshes/hokuyo.dae" />
+      </geometry>
+    </visual>
+    <collision>
+      <origin xyz="0.0 0.0 0.0" rpy="0.0 0.0 0.0"/>
+      <geometry>
+        <box size="0.1 0.1 0.1"/>
       </geometry>
     </collision>
@@ -117,3 +169,14 @@
     <child link="chassis" />
  </joint>
+ <joint name="camera_name" type="fixed">
+   <origin xyz="0.2 0.0 0.0" rpy="0.0 0.0 0.0"/>
+   <parent link="chassis"/>
+   <child link="camera"/>
+   <axis xyz="0 1 0"/>
+ </joint>
+<joint name="hokuyo_joint" type="fixed">
+  <origin xyz="0.15 0.0 0.1" rpy="0.0 0.0 0.0"/>
+  <parent link="chassis"/>
+  <child link="hokuyo"/>
+</joint>
 </robot>

Commit message: gazebo plugins

File: src/my_robot/urdf/my_robot.xacro (robot description, xacro)
@@ -1,4 +1,5 @@
 <?xml version='1.0'?>
 <robot name="my_robot" xmlns:xacro="http://www.ros.org/wiki/xacro">
+  <xacro:include filename="$(find my_robot)/urdf/my_robot.gazebo" />
   <material name="blue">
     <color rgba="0 0 0.8 1"/>
@@ -164,19 +165,19 @@
     <dynamics damping="1.0" friction="1.0"/>
   </joint>
-<joint name="robot_footprint_joint" type="fixed">
+  <joint name="robot_footprint_joint" type="fixed">
     <origin xyz="0 0 0" rpy="0 0 0" />
     <parent link="robot_footprint"/>
     <child link="chassis" />
- </joint>
- <joint name="camera_name" type="fixed">
+  </joint>
+  <joint name="camera_name" type="fixed">
    <origin xyz="0.2 0.0 0.0" rpy="0.0 0.0 0.0"/>
    <parent link="chassis"/>
    <child link="camera"/>
    <axis xyz="0 1 0"/>
- </joint>
-<joint name="hokuyo_joint" type="fixed">
-  <origin xyz="0.15 0.0 0.1" rpy="0.0 0.0 0.0"/>
-  <parent link="chassis"/>
-  <child link="hokuyo"/>
-</joint>
+  </joint>
+  <joint name="hokuyo_joint" type="fixed">
+    <origin xyz="0.15 0.0 0.1" rpy="0.0 0.0 0.0"/>
+    <parent link="chassis"/>
+    <child link="hokuyo"/>
+  </joint>
 </robot>

Commit message: RViz Integration

File: src/my_robot/urdf/my_robot.xacro (robot description, xacro)
@@ -61,4 +61,7 @@
     </visual>
   </link>
+  <gazebo reference = "chassis">
+    <material> Gazebo/Blue </material>
+  </gazebo>
   <link name="left_wheel">
 	  <inertial>
@@ -85,4 +88,7 @@
     </collision>
   </link>
+  <gazebo reference = "left_wheel">
+    <material> Gazebo/Green </material>
+  </gazebo>
   <link name="right_wheel">
 	  <inertial>
@@ -109,4 +115,7 @@
     </collision>
   </link>
+  <gazebo reference = "right_wheel">
+    <material> Gazebo/Green </material>
+  </gazebo>
   <link name="camera">
     <box_inertia x="0.05" y="0.05" z="0.05" m="0.1" />
@@ -130,4 +139,7 @@
     </collision>
   </link>
+  <gazebo reference = "camera">
+    <material> Gazebo/Red </material>
+  </gazebo>
   <link name="hokuyo">
     <inertial>

Commit message: robot modified 0.5

File: src/my_robot/urdf/my_robot.xacro (robot description, xacro)
@@ -162,5 +162,5 @@
   </link>
   <joint type="continuous" name="left_wheel_hinge">
-    <origin xyz="0 0.15 0" rpy="0 0 0"/>
+    <origin xyz="-0.15 0.15 0" rpy="0 0 0"/>
     <child link="left_wheel"/>
     <parent link="chassis"/>
@@ -170,5 +170,5 @@
   </joint>
   <joint type="continuous" name="right_wheel_hinge">
-    <origin xyz="0 -0.15 0" rpy="0 0 0"/>
+    <origin xyz="-0.15 -0.15 0" rpy="0 0 0"/>
     <child link="right_wheel"/>
     <parent link="chassis"/>

Commit message: robot modify 2

File: src/my_robot/urdf/my_robot.xacro (robot description, xacro)
@@ -26,5 +26,5 @@
       <origin xyz="0 0 0" rpy=" 0 0 0"/>
       <geometry>
-        <box size=".4 .2 .1"/>
+        <box size=".3 .2 .1"/>
       </geometry>
     </collision>
@@ -32,22 +32,10 @@
       <origin xyz="0 0 0" rpy=" 0 0 0"/>
       <geometry>
-        <box size=".4 .2 .1"/>
+        <box size=".3 .2 .1"/>
       </geometry>
       <material name="blue"/>
     </visual>
-    <collision name='back_caster_collision'>
-      <origin xyz="-0.15 0 -0.05" rpy=" 0 0 0"/>
-      <geometry>
-        <sphere radius="0.0499"/>
-      </geometry>
-    </collision>
-    <visual name='back_caster_visual'>
-      <origin xyz="-0.15 0 -0.05" rpy=" 0 0 0"/>
-      <geometry>
-        <sphere radius="0.05"/>
-      </geometry>
-    </visual>
     <collision name='front_caster_collision'>
-      <origin xyz="0.15 0 -0.05" rpy=" 0 0 0"/>
+      <origin xyz="0.1 0 -0.05" rpy=" 0 0 0"/>
       <geometry>
         <sphere radius="0.0499"/>
@@ -55,5 +43,5 @@
     </collision>
     <visual name='front_caster_visual'>
-      <origin xyz="0.15 0 -0.05" rpy=" 0 0 0"/>
+      <origin xyz="0.1 0 -0.05" rpy=" 0 0 0"/>
       <geometry>
         <sphere radius="0.05"/>
@@ -66,5 +54,5 @@
   <link name="left_wheel">
 	  <inertial>
-    	<mass value="5.0"/>
+    	<mass value="2.5"/>
     	<origin xyz="0.0 0 0" rpy=" 0 1.5707 1.5707"/>
     	<inertia
@@ -162,5 +150,5 @@
   </link>
   <joint type="continuous" name="left_wheel_hinge">
-    <origin xyz="-0.15 0.15 0" rpy="0 0 0"/>
+    <origin xyz="-0.12 0.15 0" rpy="0 0 0"/>
     <child link="left_wheel"/>
     <parent link="chassis"/>
@@ -170,5 +158,5 @@
   </joint>
   <joint type="continuous" name="right_wheel_hinge">
-    <origin xyz="-0.15 -0.15 0" rpy="0 0 0"/>
+    <origin xyz="-0.12 -0.15 0" rpy="0 0 0"/>
     <child link="right_wheel"/>
     <parent link="chassis"/>
@@ -183,5 +171,5 @@
   </joint>
   <joint name="camera_name" type="fixed">
-   <origin xyz="0.2 0.0 0.0" rpy="0.0 0.0 0.0"/>
+   <origin xyz="0.15 0.0 0.0" rpy="0.0 0.0 0.0"/>
    <parent link="chassis"/>
    <child link="camera"/>
@@ -189,5 +177,5 @@
   </joint>
   <joint name="hokuyo_joint" type="fixed">
-    <origin xyz="0.15 0.0 0.1" rpy="0.0 0.0 0.0"/>
+    <origin xyz="0.1 0.0 0.1" rpy="0.0 0.0 0.0"/>
     <parent link="chassis"/>
     <child link="hokuyo"/>

Commit message: ready for test

File: src/my_robot/urdf/my_robot.xacro (robot description, xacro)
@@ -26,5 +26,5 @@
       <origin xyz="0 0 0" rpy=" 0 0 0"/>
       <geometry>
-        <box size=".3 .2 .1"/>
+        <box size=".3 .15 .1"/>
       </geometry>
     </collision>
@@ -32,7 +32,19 @@
       <origin xyz="0 0 0" rpy=" 0 0 0"/>
       <geometry>
-        <box size=".3 .2 .1"/>
+        <cylinder radius="0.17" length="0.1"/>
       </geometry>
       <material name="blue"/>
+    </visual>
+    <collision name='back_caster_collision'>
+      <origin xyz="-0.1 0 -0.05" rpy=" 0 0 0"/>
+      <geometry>
+        <sphere radius="0.0499"/>
+      </geometry>
+    </collision>
+    <visual name='back_caster_visual'>
+      <origin xyz="-0.1 0 -0.05" rpy=" 0 0 0"/>
+      <geometry>
+        <sphere radius="0.05"/>
+      </geometry>
     </visual>
     <collision name='front_caster_collision'>
@@ -54,5 +66,5 @@
   <link name="left_wheel">
 	  <inertial>
-    	<mass value="2.5"/>
+    	<mass value="5.0"/>
     	<origin xyz="0.0 0 0" rpy=" 0 1.5707 1.5707"/>
     	<inertia
@@ -65,5 +77,5 @@
       <origin xyz="0 0 0" rpy=" 0 1.5707 1.5707"/>
       <geometry>
-        <cylinder radius="0.1" length="0.05"/>
+        <cylinder radius="0.06" length="0.05"/>
       </geometry>
       <material name="green"/>
@@ -72,5 +84,5 @@
       <origin xyz="0 0 0" rpy=" 0 1.5707 1.5707"/>
       <geometry>
-        <cylinder radius="0.1" length="0.05"/>
+        <cylinder radius="0.06" length="0.05"/>
       </geometry>
     </collision>
@@ -92,5 +104,5 @@
       <origin xyz="0 0 0" rpy=" 0 1.5707 1.5707"/>
       <geometry>
-        <cylinder radius="0.1" length="0.05"/>
+        <cylinder radius="0.06" length="0.05"/>
       </geometry>
       <material name="green"/>
@@ -99,5 +111,5 @@
       <origin xyz="0 0 0" rpy=" 0 1.5707 1.5707"/>
       <geometry>
-        <cylinder radius="0.1" length="0.05"/>
+        <cylinder radius="0.06" length="0.05"/>
       </geometry>
     </collision>
@@ -150,5 +162,5 @@
   </link>
   <joint type="continuous" name="left_wheel_hinge">
-    <origin xyz="-0.12 0.15 0" rpy="0 0 0"/>
+    <origin xyz="0 0.1 -0.04" rpy="0 0 0"/>
     <child link="left_wheel"/>
     <parent link="chassis"/>
@@ -158,5 +170,5 @@
   </joint>
   <joint type="continuous" name="right_wheel_hinge">
-    <origin xyz="-0.12 -0.15 0" rpy="0 0 0"/>
+    <origin xyz="0 -0.1 -0.04" rpy="0 0 0"/>
     <child link="right_wheel"/>
     <parent link="chassis"/>
